Commit message: IMU rotated

File: sam_description/urdf/sam_auv_base.urdf.xacro (robot description, xacro)
@@ -14,4 +14,5 @@
 <robot xmlns:xacro="http://www.ros.org/wiki/xacro" >
   <!-- Properties -->
+  <xacro:property name="simulation" default="false"/>
   <xacro:property name="mass" value="30.48"/>
   <xacro:property name="length" value="1.7"/>
@@ -26,4 +27,5 @@
   <xacro:property name="shaft_mesh_file" value="file://$(find sam_description)/mesh/sam_shaft.dae"/>
   <xacro:property name="propeller_cover_mesh_file" value="file://$(find sam_description)/mesh/sam_cover.dae"/>
+  <xacro:property name="M_PI" value="3.1415926535897931" />
   <!-- Macro for the inertial properties of a box -->
   <xacro:macro name="sam_box_inertial" params="x y z mass *origin">
@@ -179,4 +181,32 @@
       <limit upper="0" lower="0" effort="0" velocity="0" />
     </joint>
+    <!-- <xacro:if value="${simulation == 'false'}"/> -->
+      <!--IMU -->
+      <link name="${namespace}/imu_link">
+        <inertial>
+          <mass value="0.001"/>
+          <origin rpy="0 0 0" xyz="0 0 0"/>
+          <inertia ixx="0.0001" ixy="0" ixz="0" iyy="0.000001" iyz="0" izz="0.0001"/>
+        </inertial>
+        <visual>
+          <origin rpy="0 0 0" xyz="0 0 0"/>
+          <geometry>
+            <box size="0.01 0.01 0.01"/>
+          </geometry>
+          <material name="red"/>
+        </visual>
+        <collision>
+          <origin rpy="0 0 0" xyz="0 0 0"/>
+          <geometry>
+            <box size="0.01 0.01 0.01"/>
+          </geometry>
+        </collision>
+      </link>
+      <joint name="${namespace}/imu_joint" type="fixed">
+        <origin xyz="0.0 0 -0.03" rpy="0 ${M_PI/2} 0" />
+        <parent link="${namespace}/base_link"/>
+        <child link="${namespace}/imu_link"/>
+      </joint>
+    <!-- </xacro:if> -->
   </xacro:macro>
 </robot>

Commit message: Moved base_link to com

File: sam_description/urdf/sam_auv_base.urdf.xacro (robot description, xacro)
@@ -14,12 +14,14 @@
 <robot xmlns:xacro="http://www.ros.org/wiki/xacro" >
   <!-- Properties -->
-  <xacro:property name="simulation" default="false"/>
-  <xacro:property name="mass" value="30.48"/>
-  <xacro:property name="length" value="1.7"/>
-  <xacro:property name="diameter" value="0.19"/>
+  <xacro:property name="mass" value="14"/>
+  <xacro:property name="length" value="1.33"/>
+  <xacro:property name="diameter" value="0.125"/>
   <xacro:property name="radius" value="${diameter*0.5}"/>
+  <xacro:property name="cylinder_length" value="1.094"/>
+  <xacro:property name="base_link_shift" value="${0.627 - cylinder_length}"/>
   <!-- <xacro:property name="volume" value="${length*pi*radius*radius}"/> -->
-  <xacro:property name="volume" value="0.030431864"/>
-  <xacro:property name="cob" value="0 0 0.0196"/>
+  <xacro:property name="volume" value="0.014"/>
+  <xacro:property name="cob" value="0 0 0.03"/>
+  <xacro:property name="com" value="0 0 0"/>
   <xacro:property name="rho" value="1025.0"/>
   <xacro:property name="visual_mesh_file" value="file://$(find sam_description)/mesh/sam_body.dae"/>
@@ -41,5 +43,5 @@
     <link name="${namespace}/base_link">
       <visual>
-        <origin xyz="0 0 0" rpy="0 0 0"/>
+        <origin xyz="${-base_link_shift} 0 0" rpy="0 0 0"/>
         <geometry>
           <mesh filename="${visual_mesh_file}" scale="1 1 1" />
@@ -54,13 +56,13 @@
       <inertial>
         <mass value="${mass}" />
-        <origin xyz="0 0 0" rpy="0 0 0"/>
-        <inertia ixx="0.177" ixy="0" ixz="0"
-                 iyy="3.45" iyz="0"
-                 izz="3.45" />
+        <origin xyz="${com}" rpy="0 0 0"/>
+        <inertia ixx="0.0294" ixy="0" ixz="0"
+                 iyy="1.6202" iyz="0"
+                 izz="1.6202" />
       </inertial>
     </link>
 	<!-- Shaft -->
     <joint name="${namespace}/shaft_joint1" type="revolute">
-      <origin xyz="-1.045 0 0" rpy="0 0 0" />
+      <origin xyz="${-1.045 - base_link_shift} 0 0" rpy="0 0 0" />
       <axis xyz="0 0 1"/>
       <parent link="${namespace}/base_link"/>

Commit message: Added flag for simulation/real robot launch

File: sam_description/urdf/sam_auv_base.urdf.xacro (robot description, xacro)
@@ -29,4 +29,5 @@
   <xacro:property name="shaft_mesh_file" value="file://$(find sam_description)/mesh/sam_shaft.dae"/>
   <xacro:property name="propeller_cover_mesh_file" value="file://$(find sam_description)/mesh/sam_cover.dae"/>
+  <xacro:property name="simulation" default="false"/>
   <xacro:property name="M_PI" value="3.1415926535897931" />
   <!-- Macro for the inertial properties of a box -->
@@ -183,5 +184,5 @@
       <limit upper="0" lower="0" effort="0" velocity="0" />
     </joint>
-    <!-- <xacro:if value="${simulation == 'false'}"/> -->
+    <xacro:unless value="${simulation}">
       <!--IMU -->
       <link name="${namespace}/imu_link">
@@ -206,9 +207,9 @@
       </link>
       <joint name="${namespace}/imu_joint" type="fixed">
-        <origin xyz="0.0 0 -0.03" rpy="0 ${M_PI/2} 0" />
+        <origin xyz="0.0 0 -0.03" rpy="0 -${M_PI/2} 0" />
         <parent link="${namespace}/base_link"/>
         <child link="${namespace}/imu_link"/>
       </joint>
-    <!-- </xacro:if> -->
+    </xacro:unless>
   </xacro:macro>
 </robot>

Commit message: Added joints for DVL and pressure sensor

File: sam_description/urdf/sam_auv_base.urdf.xacro (robot description, xacro)
@@ -19,5 +19,5 @@
   <xacro:property name="radius" value="${diameter*0.5}"/>
   <xacro:property name="cylinder_length" value="1.094"/>
-  <xacro:property name="base_link_shift" value="${0.627 - cylinder_length}"/>
+  <xacro:property name="base_link_shift" value="${0.737 - cylinder_length}"/>
   <!-- <xacro:property name="volume" value="${length*pi*radius*radius}"/> -->
   <xacro:property name="volume" value="0.014"/>
@@ -184,4 +184,5 @@
       <limit upper="0" lower="0" effort="0" velocity="0" />
     </joint>
+    <!-- Sensors  -->
     <xacro:unless value="${simulation}">
       <!--IMU -->
@@ -207,7 +208,133 @@
       </link>
       <joint name="${namespace}/imu_joint" type="fixed">
-        <origin xyz="0.0 0 -0.03" rpy="0 -${M_PI/2} 0" />
+        <origin xyz="0.273 0 -0.03" rpy="0 -${M_PI/2} 0" />
         <parent link="${namespace}/base_link"/>
         <child link="${namespace}/imu_link"/>
+      </joint>
+      <!-- DVL: three heads + main sensor frame -->
+      <link name="${namespace}/dvl_link">
+        <inertial>
+          <mass value="0.001"/>
+          <origin rpy="0 0 0" xyz="0 0 0"/>
+          <inertia ixx="0.0001" ixy="0" ixz="0" iyy="0.000001" iyz="0" izz="0.0001"/>
+        </inertial>
+        <visual>
+          <origin rpy="0 0 0" xyz="0 0 0"/>
+          <geometry>
+            <box size="0.01 0.01 0.01"/>
+          </geometry>
+          <material name="blue"/>
+        </visual>
+        <collision>
+          <origin rpy="0 0 0" xyz="0 0 0"/>
+          <geometry>
+            <box size="0.01 0.01 0.01"/>
+          </geometry>
+        </collision>
+      </link>
+      <joint name="${namespace}/dvl_joint" type="fixed">
+        <origin xyz="0.530 0 -0.03" rpy="0 0 0" />
+        <parent link="${namespace}/base_link"/>
+        <child link="${namespace}/dvl_link"/>
+      </joint>
+      <link name="${namespace}/dvl_port_link">
+        <inertial>
+          <mass value="0.001"/>
+          <origin rpy="0 0 0" xyz="0 0 0"/>
+          <inertia ixx="0.0001" ixy="0" ixz="0" iyy="0.000001" iyz="0" izz="0.0001"/>
+        </inertial>
+        <visual>
+          <origin rpy="0 0 0" xyz="0 0 0"/>
+          <geometry>
+            <box size="0.01 0.01 0.01"/>
+          </geometry>
+          <material name="blue"/>
+        </visual>
+        <collision>
+          <origin rpy="0 0 0" xyz="0 0 0"/>
+          <geometry>
+            <box size="0.01 0.01 0.01"/>
+          </geometry>
+        </collision>
+      </link>
+      <joint name="${namespace}/dvl_port_joint" type="fixed">
+        <origin xyz="0.0 0.0 0.0" rpy="0 1.22173 0.785398" />
+        <parent link="${namespace}/dvl_link"/>
+        <child link="${namespace}/dvl_port_link"/>
+      </joint>
+      <link name="${namespace}/dvl_down_link">
+        <inertial>
+          <mass value="0.001"/>
+          <origin rpy="0 0 0" xyz="0 0 0"/>
+          <inertia ixx="0.0001" ixy="0" ixz="0" iyy="0.000001" iyz="0" izz="0.0001"/>
+        </inertial>
+        <visual>
+          <origin rpy="0 0 0" xyz="0 0 0"/>
+          <geometry>
+            <box size="0.01 0.01 0.01"/>
+          </geometry>
+          <material name="blue"/>
+        </visual>
+        <collision>
+          <origin rpy="0 0 0" xyz="0 0 0"/>
+          <geometry>
+            <box size="0.01 0.01 0.01"/>
+          </geometry>
+        </collision>
+      </link>
+      <joint name="${namespace}/dvl_down_joint" type="fixed">
+        <origin xyz="0.0 0.0 0.0" rpy="0 ${M_PI/2} 0" />
+        <parent link="${namespace}/dvl_link"/>
+        <child link="${namespace}/dvl_down_link"/>
+      </joint>
+       <link name="${namespace}/dvl_starboard_link">
+        <inertial>
+          <mass value="0.001"/>
+          <origin rpy="0 0 0" xyz="0 0 0"/>
+          <inertia ixx="0.0001" ixy="0" ixz="0" iyy="0.000001" iyz="0" izz="0.0001"/>
+        </inertial>
+        <visual>
+          <origin rpy="0 0 0" xyz="0 0 0"/>
+          <geometry>
+            <box size="0.01 0.01 0.01"/>
+          </geometry>
+          <material name="blue"/>
+        </visual>
+        <collision>
+          <origin rpy="0 0 0" xyz="0 0 0"/>
+          <geometry>
+            <box size="0.01 0.01 0.01"/>
+          </geometry>
+        </collision>
+      </link>
+      <joint name="${namespace}/dvl_starboard_joint" type="fixed">
+        <origin xyz="0. 0.0 0.0" rpy="0 1.22173 -0.785398" />
+        <parent link="${namespace}/dvl_link"/>
+        <child link="${namespace}/dvl_starboard_link"/>
+      </joint>
+      <link name="${namespace}/pressure_link">
+        <inertial>
+          <mass value="0.001"/>
+          <origin rpy="0 0 0" xyz="0 0 0"/>
+          <inertia ixx="0.0001" ixy="0" ixz="0" iyy="0.000001" iyz="0" izz="0.0001"/>
+        </inertial>
+        <visual>
+          <origin rpy="0 0 0" xyz="0 0 0"/>
+          <geometry>
+            <box size="0.01 0.01 0.01"/>
+          </geometry>
+          <material name="blue"/>
+        </visual>
+        <collision>
+          <origin rpy="0 0 0" xyz="0 0 0"/>
+          <geometry>
+            <box size="0.01 0.01 0.01"/>
+          </geometry>
+        </collision>
+      </link>
+      <joint name="${namespace}/pressure_joint" type="fixed">
+        <origin xyz="-0.562 0.0 -0.03 " rpy="0 0 0" />
+        <parent link="${namespace}/base_link"/>
+        <child link="${namespace}/pressure_link"/>
       </joint>
     </xacro:unless>

Commit message: IMU frame back to original pose

File: sam_description/urdf/sam_auv_base.urdf.xacro (robot description, xacro)
@@ -208,5 +208,5 @@
       </link>
       <joint name="${namespace}/imu_joint" type="fixed">
-        <origin xyz="0.273 0 -0.03" rpy="0 -${M_PI/2} 0" />
+        <origin xyz="0.273 0 -0.03" rpy="0 0 0" />
         <parent link="${namespace}/base_link"/>
         <child link="${namespace}/imu_link"/>

Commit message: Added SBG IMU and GPS frames

File: sam_description/urdf/sam_auv_base.urdf.xacro (robot description, xacro)
@@ -19,5 +19,5 @@
   <xacro:property name="radius" value="${diameter*0.5}"/>
   <xacro:property name="cylinder_length" value="1.094"/>
-  <xacro:property name="base_link_shift" value="${0.737 - cylinder_length}"/>
+  <xacro:property name="base_link_shift" value="${0.734 - cylinder_length}"/>
   <!-- <xacro:property name="volume" value="${length*pi*radius*radius}"/> -->
   <xacro:property name="volume" value="0.014"/>
@@ -186,5 +186,57 @@
     <!-- Sensors  -->
     <xacro:unless value="${simulation}">
-      <!--IMU -->
+      <!--GPS -->
+      <link name="${namespace}/gps_link">
+        <inertial>
+          <mass value="0.001"/>
+          <origin rpy="0 0 0" xyz="0 0 0"/>
+          <inertia ixx="0.0001" ixy="0" ixz="0" iyy="0.000001" iyz="0" izz="0.0001"/>
+        </inertial>
+        <visual>
+          <origin rpy="0 0 0" xyz="0 0 0"/>
+          <geometry>
+            <box size="0.01 0.01 0.01"/>
+          </geometry>
+          <material name="red"/>
+        </visual>
+        <collision>
+          <origin rpy="0 0 0" xyz="0 0 0"/>
+          <geometry>
+            <box size="0.01 0.01 0.01"/>
+          </geometry>
+        </collision>
+      </link>
+      <joint name="${namespace}/gps_joint" type="fixed">
+        <origin xyz="0.502 0 0.0" rpy="0 0 0" />
+        <parent link="${namespace}/base_link"/>
+        <child link="${namespace}/gps_link"/>
+      </joint>
+      <!--SBG IMU -->
+      <link name="${namespace}/sbg_link">
+        <inertial>
+          <mass value="0.001"/>
+          <origin rpy="0 0 0" xyz="0 0 0"/>
+          <inertia ixx="0.0001" ixy="0" ixz="0" iyy="0.000001" iyz="0" izz="0.0001"/>
+        </inertial>
+        <visual>
+          <origin rpy="0 0 0" xyz="0 0 0"/>
+          <geometry>
+            <box size="0.01 0.01 0.01"/>
+          </geometry>
+          <material name="red"/>
+        </visual>
+        <collision>
+          <origin rpy="0 0 0" xyz="0 0 0"/>
+          <geometry>
+            <box size="0.01 0.01 0.01"/>
+          </geometry>
+        </collision>
+      </link>
+      <joint name="${namespace}/sbg_joint" type="fixed">
+        <origin xyz="0.472 0 0.03" rpy="0 0 0" />
+        <parent link="${namespace}/base_link"/>
+        <child link="${namespace}/sbg_link"/>
+      </joint>
+      <!--STIM IMU -->
       <link name="${namespace}/imu_link">
         <inertial>
@@ -208,5 +260,5 @@
       </link>
       <joint name="${namespace}/imu_joint" type="fixed">
-        <origin xyz="0.273 0 -0.03" rpy="0 0 0" />
+        <origin xyz="0.192 0 -0.03" rpy="0 0 0" />
         <parent link="${namespace}/base_link"/>
         <child link="${namespace}/imu_link"/>

Commit message: Rotated SBG for ENU convention

File: sam_description/urdf/sam_auv_base.urdf.xacro (robot description, xacro)
@@ -234,5 +234,5 @@
       </link>
       <joint name="${namespace}/sbg_joint" type="fixed">
-        <origin xyz="0.472 0 0.03" rpy="0 0 0" />
+        <origin xyz="0.472 0 0.03" rpy="0 0 -${M_PI/2}" />
         <parent link="${namespace}/base_link"/>
         <child link="${namespace}/sbg_link"/>

Commit message: Changed SBG frame. All tested now

File: sam_description/urdf/sam_auv_base.urdf.xacro (robot description, xacro)
@@ -234,5 +234,5 @@
       </link>
       <joint name="${namespace}/sbg_joint" type="fixed">
-        <origin xyz="0.472 0 0.03" rpy="0 0 -${M_PI/2}" />
+        <origin xyz="0.472 0 0.03" rpy="0 0 0" />
         <parent link="${namespace}/base_link"/>
         <child link="${namespace}/sbg_link"/>

Commit message: Added camera down link. Missing the others

File: sam_description/urdf/sam_auv_base.urdf.xacro (robot description, xacro)
@@ -264,4 +264,31 @@
         <child link="${namespace}/imu_link"/>
       </joint>
+      <!-- Cameras: three cams + main sensor frame -->
+      <!-- TODO: add missing ones -->
+      <link name="${namespace}/camera_down_link">
+        <inertial>
+          <mass value="0.001"/>
+          <origin rpy="0 0 0" xyz="0 0 0"/>
+          <inertia ixx="0.0001" ixy="0" ixz="0" iyy="0.000001" iyz="0" izz="0.0001"/>
+        </inertial>
+        <visual>
+          <origin rpy="0 0 0" xyz="0 0 0"/>
+          <geometry>
+            <box size="0.01 0.01 0.01"/>
+          </geometry>
+          <material name="blue"/>
+        </visual>
+        <collision>
+          <origin rpy="0 0 0" xyz="0 0 0"/>
+          <geometry>
+            <box size="0.01 0.01 0.01"/>
+          </geometry>
+        </collision>
+      </link>
+      <joint name="${namespace}/camera_down_joint" type="fixed">
+        <origin xyz="0.530 0 -0.03" rpy="0 ${M_PI/2} 0" />
+        <parent link="${namespace}/base_link"/>
+        <child link="${namespace}/camera_down_link"/>
+      </joint>
       <!-- DVL: three heads + main sensor frame -->
       <link name="${namespace}/dvl_link">

Commit message: Added lateral cameras frames

File: sam_description/urdf/sam_auv_base.urdf.xacro (robot description, xacro)
@@ -291,4 +291,54 @@
         <child link="${namespace}/camera_down_link"/>
       </joint>
+      <link name="${namespace}/camera_front_left_link">
+        <inertial>
+          <mass value="0.001"/>
+          <origin rpy="0 0 0" xyz="0 0 0"/>
+          <inertia ixx="0.0001" ixy="0" ixz="0" iyy="0.000001" iyz="0" izz="0.0001"/>
+        </inertial>
+        <visual>
+          <origin rpy="0 0 0" xyz="0 0 0"/>
+          <geometry>
+            <box size="0.01 0.01 0.01"/>
+          </geometry>
+          <material name="blue"/>
+        </visual>
+        <collision>
+          <origin rpy="0 0 0" xyz="0 0 0"/>
+          <geometry>
+            <box size="0.01 0.01 0.01"/>
+          </geometry>
+        </collision>
+      </link>
+      <joint name="${namespace}/camera_front_left_joint" type="fixed">
+        <origin xyz="1.313 0.048 -0.007" rpy="1.3 3.1416 2.3416" />
+        <parent link="${namespace}/base_link"/>
+        <child link="${namespace}/camera_front_left_link"/>
+      </joint>
+      <link name="${namespace}/camera_front_right_link">
+        <inertial>
+          <mass value="0.001"/>
+          <origin rpy="0 0 0" xyz="0 0 0"/>
+          <inertia ixx="0.0001" ixy="0" ixz="0" iyy="0.000001" iyz="0" izz="0.0001"/>
+        </inertial>
+        <visual>
+          <origin rpy="0 0 0" xyz="0 0 0"/>
+          <geometry>
+            <box size="0.01 0.01 0.01"/>
+          </geometry>
+          <material name="blue"/>
+        </visual>
+        <collision>
+          <origin rpy="0 0 0" xyz="0 0 0"/>
+          <geometry>
+            <box size="0.01 0.01 0.01"/>
+          </geometry>
+        </collision>
+      </link>
+      <joint name="${namespace}/camera_front_right_joint" type="fixed">
+        <origin xyz="1.313 -0.048 -0.007" rpy="1.3 3.1416 0.8" />
+        <parent link="${namespace}/base_link"/>
+        <child link="${namespace}/camera_front_right_link"/>
+      </joint>
       <!-- DVL: three heads + main sensor frame -->
       <link name="${namespace}/dvl_link">
