Commit message: Added SGB link to urdf

File: sam_description/urdf/sam_auv.urdf.xacro (robot description, xacro)
@@ -23,4 +23,8 @@
   <link name="$(arg robot_namespace)/imu_link">
   </link>
+  <link name="$(arg robot_namespace)/sbg_link">
+  </link>
+<!--   <link name="$(arg robot_namespace)/mag_link">
+  </link> -->
   <link name="$(arg robot_namespace)/gps_link">
   </link>
@@ -51,4 +55,15 @@
     <origin rpy="0.0 0.0 0.0" xyz="0.9 0.0 0.0"/>
   </joint>
+  <joint name="$(arg robot_namespace)/sbg_joint" type="fixed">
+    <parent link="$(arg robot_namespace)/base_link"/>
+    <child link="$(arg robot_namespace)/sbg_link"/>
+    <origin rpy="0.0 0.0 0.0" xyz="0.472 0 0.03"/>
+  </joint>
+    <!-- Compass doesn't seem to have a ROS parser -->
+<!--   <joint name="$(arg robot_namespace)/mag_joint" type="fixed">
+    <parent link="$(arg robot_namespace)/base_link"/>
+    <child link="$(arg robot_namespace)/mag_link"/>
+    <origin rpy="0.0 0.0 0.0" xyz="0.472 0 0.03"/>
+  </joint> -->
   <joint name="$(arg robot_namespace)/gps_joint" type="fixed">
     <parent link="$(arg robot_namespace)/base_link"/>

Commit message: Update sam_auv urdf file to comply with most recent real-life SAM

File: sam_description/urdf/sam_auv.urdf.xacro (robot description, xacro)
@@ -1,89 +1,56 @@
 <?xml version="1.0"?>
 <robot name="sam_auv" xmlns:xacro="http://www.ros.org/wiki/xacro">
-  <!-- ECA 5E Micro mnipulator -->
-  <!-- links -->
+  <!-- Meshes. -->
+  <xacro:property name="visual_mesh_file" value="file://$(find sam_description)/mesh/SAM_HULL.dae"/>
+  <xacro:property name="prop_nozzle" value="file://$(find sam_description)/mesh/SAM_NOZZLE.dae"/>
+  <xacro:property name="front_prop" value="file://$(find sam_description)/mesh/SAM_FRONTPROP.dae"/>
+  <xacro:property name="back_prop" value="file://$(find sam_description)/mesh/SAM_BACKPROP.dae"/>
+  <!-- Links. -->
   <link name="$(arg robot_namespace)/base_link">
-  </link>
-  <link name="$(arg robot_namespace)/thruster_yaw_link">
+    <visual>
+      <origin xyz="0 0 0" rpy="0 0 0"/>
+      <geometry>
+        <mesh filename="${visual_mesh_file}" scale="1 1 1"/>
+      </geometry>
+    </visual>
   </link>
   <link name="$(arg robot_namespace)/thruster_link">
+    <visual>
+      <origin xyz="0 0 0" rpy="0 0 0"/>
+      <geometry>
+        <mesh filename="${prop_nozzle}" scale="1 1 1"/>
+      </geometry>
+    </visual>
   </link>
-  <link name="$(arg robot_namespace)/battery_link">
+  <link name="$(arg robot_namespace)/front_prop_link">
+    <visual>
+      <origin xyz="0 0 0" rpy="0 0 0"/>
+      <geometry>
+        <mesh filename="${front_prop}" scale="1 1 1"/>
+      </geometry>
+    </visual>
   </link>
-  <link name="$(arg robot_namespace)/tcg1_link">
+  <link name="$(arg robot_namespace)/back_prop_link">
+    <visual>
+      <origin xyz="0 0 0" rpy="0 0 0"/>
+      <geometry>
+        <mesh filename="${back_prop}" scale="1 1 1"/>
+      </geometry>
+    </visual>
   </link>
-  <link name="$(arg robot_namespace)/tcg2_link">
-  </link>
-  <link name="$(arg robot_namespace)/multibeam_down_link">
-  </link>
-  <link name="$(arg robot_namespace)/pressure_link">
-  </link>
-  <link name="$(arg robot_namespace)/dvl_link">
-  </link>
-  <link name="$(arg robot_namespace)/imu_link">
-  </link>
-  <link name="$(arg robot_namespace)/sbg_link">
-  </link>
-<!--   <link name="$(arg robot_namespace)/mag_link">
-  </link> -->
-  <link name="$(arg robot_namespace)/gps_link">
-  </link>
-  <link name="$(arg robot_namespace)/camera_down_link">
-  </link>
-  <link name="$(arg robot_namespace)/camera_front_right_link">
-  </link>
-  <link name="$(arg robot_namespace)/camera_front_left_link">
-  </link>
-  <joint name="$(arg robot_namespace)/multibeam_down_joint" type="fixed">
-    <parent link="$(arg robot_namespace)/base_link"/>
-    <child link="$(arg robot_namespace)/multibeam_down_link"/>
-    <origin rpy="0.0 1.5707 0.0" xyz="1.20 0.0 -0.07"/>
-  </joint>
-  <joint name="$(arg robot_namespace)/pressure_joint" type="fixed">
-    <parent link="$(arg robot_namespace)/base_link"/>
-    <child link="$(arg robot_namespace)/pressure_link"/>
-    <origin rpy="0.0 0.0 0.0" xyz="0.3 0.0 0.07"/>
-  </joint>
-  <joint name="$(arg robot_namespace)/dvl_joint" type="fixed">
-    <parent link="$(arg robot_namespace)/base_link"/>
-    <child link="$(arg robot_namespace)/dvl_link"/>
-    <origin rpy="0.0 0.0 0.0" xyz="1.25 0.0 -0.07"/>
-  </joint>
-  <joint name="$(arg robot_namespace)/imu_joint" type="fixed">
-    <parent link="$(arg robot_namespace)/base_link"/>
-    <child link="$(arg robot_namespace)/imu_link"/>
-    <origin rpy="0.0 0.0 0.0" xyz="0.9 0.0 0.0"/>
-  </joint>
-  <joint name="$(arg robot_namespace)/sbg_joint" type="fixed">
-    <parent link="$(arg robot_namespace)/base_link"/>
-    <child link="$(arg robot_namespace)/sbg_link"/>
-    <origin rpy="0.0 0.0 0.0" xyz="0.472 0 0.03"/>
-  </joint>
-    <!-- Compass doesn't seem to have a ROS parser -->
-<!--   <joint name="$(arg robot_namespace)/mag_joint" type="fixed">
-    <parent link="$(arg robot_namespace)/base_link"/>
-    <child link="$(arg robot_namespace)/mag_link"/>
-    <origin rpy="0.0 0.0 0.0" xyz="0.472 0 0.03"/>
-  </joint> -->
-  <joint name="$(arg robot_namespace)/gps_joint" type="fixed">
-    <parent link="$(arg robot_namespace)/base_link"/>
-    <child link="$(arg robot_namespace)/gps_link"/>
-    <origin rpy="0.0 1.5707 0.0" xyz="1.2 0.0 0.08"/>
-  </joint>
-  <joint name="$(arg robot_namespace)/camera_down_joint" type="fixed">
-    <parent link="$(arg robot_namespace)/base_link"/>
-    <child link="$(arg robot_namespace)/camera_down_link"/>
-    <origin rpy="3.1416 0.0 -1.5707" xyz="1.15 0.0 -0.07"/>
-  </joint>
-  <joint name="$(arg robot_namespace)/camera_front_right_joint" type="fixed">
-    <parent link="$(arg robot_namespace)/base_link"/>
-    <child link="$(arg robot_namespace)/camera_front_right_link"/>
-    <origin rpy="1.3 3.1416 2.3416" xyz="1.32 0.05 0.005"/>
-  </joint>
-  <joint name="$(arg robot_namespace)/camera_front_left_joint" type="fixed">
-    <parent link="$(arg robot_namespace)/base_link"/>
-    <child link="$(arg robot_namespace)/camera_front_left_link"/>
-    <origin rpy="1.3 3.1416 0.8" xyz="1.32 -0.05 0.005"/>
-  </joint>
+  <link name="$(arg robot_namespace)/thruster_yaw_link"/>
+  <link name="$(arg robot_namespace)/battery_link"/>
+  <link name="$(arg robot_namespace)/tcg1_link"/>
+  <link name="$(arg robot_namespace)/tcg2_link"/>
+  <link name="$(arg robot_namespace)/pressure_link"/>
+  <link name="$(arg robot_namespace)/dvl_link"/>
+  <link name="$(arg robot_namespace)/sidescan_link"/>
+  <link name="$(arg robot_namespace)/imu_link"/>
+  <link name="$(arg robot_namespace)/sbg_link"/>
+  <link name="$(arg robot_namespace)/gps_link"/>
+  <link name="$(arg robot_namespace)/uw_gps_link"/>
+  <link name="$(arg robot_namespace)/camera_down_link"/>
+  <link name="$(arg robot_namespace)/camera_front_right_link"/>
+  <link name="$(arg robot_namespace)/camera_front_left_link"/>
   <joint name="$(arg robot_namespace)/thruster_yaw_joint" type="revolute">
     <parent link="$(arg robot_namespace)/base_link"/>
@@ -100,4 +67,67 @@
     <limit lower="-0.2" upper="0.2" velocity="0.2" effort="1.0"/>
   </joint>
+  <joint name="$(arg robot_namespace)/front_prop_joint" type="continuous">
+    <parent link="$(arg robot_namespace)/base_link"/>
+    <child link="$(arg robot_namespace)/front_prop_link"/>
+    <origin rpy="0.0 0.0 0.0" xyz="-0.056 0 0"/>
+    <axis xyz="1 0 0"/>
+  </joint>
+  <joint name="$(arg robot_namespace)/back_prop_joint" type="continuous">
+    <parent link="$(arg robot_namespace)/base_link"/>
+    <child link="$(arg robot_namespace)/back_prop_link"/>
+    <origin rpy="0.0 0.0 0.0" xyz="-0.074 0 0"/>
+    <axis xyz="1 0 0"/>
+  </joint>
+  <joint name="$(arg robot_namespace)/pressure_joint" type="fixed">
+    <parent link="$(arg robot_namespace)/base_link"/>
+    <child link="$(arg robot_namespace)/pressure_link"/>
+    <origin rpy="0.0 0.0 0.0" xyz="0.174 0.025 0.057"/>
+  </joint>
+  <joint name="$(arg robot_namespace)/dvl_joint" type="fixed">
+    <parent link="$(arg robot_namespace)/base_link"/>
+    <child link="$(arg robot_namespace)/dvl_link"/>
+    <origin rpy="0.0 0.0 0.0" xyz="1.25 0.0 -0.063"/>
+  </joint>
+  <!--Sidescan acoustic center, i.e. intersection between both sidescan centers.-->
+  <joint name="$(arg robot_namespace)/sidescan_joint" type="fixed">
+    <parent link="$(arg robot_namespace)/base_link"/>
+    <child link="$(arg robot_namespace)/sidescan_link"/>
+    <origin rpy="0.0 0.0 0.0" xyz="0.634 0.0 0.0"/>
+  </joint>
+  <joint name="$(arg robot_namespace)/imu_joint" type="fixed">
+    <parent link="$(arg robot_namespace)/base_link"/>
+    <child link="$(arg robot_namespace)/imu_link"/>
+    <origin rpy="0.0 0.0 0.0" xyz="0.917 0.0 -0.036"/>
+  </joint>
+  <joint name="$(arg robot_namespace)/sbg_joint" type="fixed">
+    <parent link="$(arg robot_namespace)/base_link"/>
+    <child link="$(arg robot_namespace)/sbg_link"/>
+    <origin rpy="0.0 0.0 0.0" xyz="1.137 0.0 0.002"/>
+  </joint>
+  <joint name="$(arg robot_namespace)/gps_joint" type="fixed">
+    <parent link="$(arg robot_namespace)/base_link"/>
+    <child link="$(arg robot_namespace)/gps_link"/>
+    <origin rpy="0.0 0.0 0.0" xyz="1.205 0.0 0.071"/>
+  </joint>
+  <joint name="$(arg robot_namespace)/uw_gps_joint" type="fixed">
+    <parent link="$(arg robot_namespace)/base_link"/>
+    <child link="$(arg robot_namespace)/uw_gps_link"/>
+    <origin rpy="0.0 0.0 0.0" xyz="0.275 0.0 0.078"/>
+  </joint>
+  <joint name="$(arg robot_namespace)/camera_down_joint" type="fixed">
+    <parent link="$(arg robot_namespace)/base_link"/>
+    <child link="$(arg robot_namespace)/camera_down_link"/>
+    <origin rpy="3.1416 0.0 -1.5707" xyz="1.1385 0.0 -0.052"/>
+  </joint>
+  <joint name="$(arg robot_namespace)/camera_front_left_joint" type="fixed">
+    <parent link="$(arg robot_namespace)/base_link"/>
+    <child link="$(arg robot_namespace)/camera_front_left_link"/>
+    <origin rpy="1.3 3.1416 2.3416" xyz="1.313 0.048 -0.007"/>
+  </joint>
+  <joint name="$(arg robot_namespace)/camera_front_right_joint" type="fixed">
+    <parent link="$(arg robot_namespace)/base_link"/>
+    <child link="$(arg robot_namespace)/camera_front_right_link"/>
+    <origin rpy="1.3 3.1416 0.8" xyz="1.313 -0.048 -0.007"/>
+  </joint>
   <joint name="$(arg robot_namespace)/lcg_joint" type="prismatic">
     <parent link="$(arg robot_namespace)/base_link"/>
@@ -110,5 +140,5 @@
     <parent link="$(arg robot_namespace)/base_link"/>
     <child link="$(arg robot_namespace)/tcg1_link"/>
-    <origin rpy="0.0 0.0 0.0" xyz="0.48 0.0 0.0"/>
+    <origin rpy="0.0 0.0 0.0" xyz="0.582 0.0 0.0"/>
     <axis xyz="1 0 0"/>
     <limit lower="-1.6" upper="1.6" velocity="0.2" effort="1.0"/>
@@ -117,5 +147,5 @@
     <parent link="$(arg robot_namespace)/base_link"/>
     <child link="$(arg robot_namespace)/tcg2_link"/>
-    <origin rpy="0.0 0.0 0.0" xyz="0.46 0.0 0.0"/>
+    <origin rpy="0.0 0.0 0.0" xyz="0.552 0.0 0.0"/>
     <axis xyz="1 0 0"/>
     <limit lower="-1.6" upper="1.6" velocity="0.2" effort="1.0"/>

Commit message: Base_link moved to cob of SAM

File: sam_description/urdf/sam_auv.urdf.xacro (robot description, xacro)
@@ -10,5 +10,5 @@
   <link name="$(arg namespace)/base_link">
     <visual>
-      <origin xyz="0 0 0" rpy="0 0 0"/>
+      <origin xyz="-0.677 0 0" rpy="0 0 0"/>
       <geometry>
         <mesh filename="${visual_mesh_file}" scale="1 1 1"/>
@@ -57,5 +57,5 @@
     <parent link="$(arg namespace)/base_link"/>
     <child link="$(arg namespace)/thruster_yaw_link"/>
-    <origin rpy="0.0 0.0 0.0" xyz="0.0 0.0 0.0"/>
+    <origin rpy="0.0 0.0 0.0" xyz="-0.677 0.0 0.0"/>
     <axis xyz="0 0 1"/>
     <limit lower="-0.2" upper="0.2" velocity="0.2" effort="1.0"/>
@@ -71,5 +71,5 @@
     <parent link="$(arg namespace)/base_link"/>
     <child link="$(arg namespace)/front_prop_link"/>
-    <origin rpy="0.0 0.0 0.0" xyz="-0.056 0 0"/>
+    <origin rpy="0.0 0.0 0.0" xyz="-0.733 0 0"/>
     <axis xyz="1 0 0"/>
   </joint>
@@ -77,5 +77,5 @@
     <parent link="$(arg namespace)/base_link"/>
     <child link="$(arg namespace)/back_prop_link"/>
-    <origin rpy="0.0 0.0 0.0" xyz="-0.074 0 0"/>
+    <origin rpy="0.0 0.0 0.0" xyz="-0.751 0 0"/>
     <axis xyz="1 0 0"/>
   </joint>
@@ -83,10 +83,10 @@
     <parent link="$(arg namespace)/base_link"/>
     <child link="$(arg namespace)/pressure_link"/>
-    <origin rpy="0.0 0.0 0.0" xyz="0.174 0.025 0.057"/>
+    <origin rpy="0.0 0.0 0.0" xyz="-0.503 0.025 0.057"/>
   </joint>
   <joint name="$(arg namespace)/dvl_joint" type="fixed">
     <parent link="$(arg namespace)/base_link"/>
     <child link="$(arg namespace)/dvl_link"/>
-    <origin rpy="0.0 0.0 0.0" xyz="1.25 0.0 -0.063"/>
+    <origin rpy="0.0 0.0 0.0" xyz="0.573 0.0 -0.063"/>
   </joint>
   <!--Sidescan acoustic center, i.e. intersection between both sidescan centers.-->
@@ -94,45 +94,45 @@
     <parent link="$(arg namespace)/base_link"/>
     <child link="$(arg namespace)/sidescan_link"/>
-    <origin rpy="0.0 0.0 0.0" xyz="0.634 0.0 0.0"/>
+    <origin rpy="0.0 0.0 0.0" xyz="-0.043 0.0 0.0"/>
   </joint>
   <joint name="$(arg namespace)/imu_joint" type="fixed">
     <parent link="$(arg namespace)/base_link"/>
     <child link="$(arg namespace)/imu_link"/>
-    <origin rpy="0.0 0.0 0.0" xyz="0.917 0.0 -0.036"/>
+    <origin rpy="0.0 0.0 0.0" xyz="0.24 0.0 -0.036"/>
   </joint>
   <joint name="$(arg namespace)/sbg_joint" type="fixed">
     <parent link="$(arg namespace)/base_link"/>
     <child link="$(arg namespace)/sbg_link"/>
-    <origin rpy="0.0 0.0 0.0" xyz="1.137 0.0 0.002"/>
+    <origin rpy="0.0 0.0 0.0" xyz="0.46 0.0 0.002"/>
   </joint>
   <joint name="$(arg namespace)/gps_joint" type="fixed">
     <parent link="$(arg namespace)/base_link"/>
     <child link="$(arg namespace)/gps_link"/>
-    <origin rpy="0.0 0.0 0.0" xyz="1.205 0.0 0.071"/>
+    <origin rpy="0.0 0.0 0.0" xyz="0.528 0.0 0.071"/>
   </joint>
   <joint name="$(arg namespace)/uw_gps_joint" type="fixed">
     <parent link="$(arg namespace)/base_link"/>
     <child link="$(arg namespace)/uw_gps_link"/>
-    <origin rpy="0.0 0.0 0.0" xyz="0.275 0.0 0.078"/>
+    <origin rpy="0.0 0.0 0.0" xyz="-0.402 0.0 0.078"/>
   </joint>
   <joint name="$(arg namespace)/camera_down_joint" type="fixed">
     <parent link="$(arg namespace)/base_link"/>
     <child link="$(arg namespace)/camera_down_link"/>
-    <origin rpy="3.1416 0.0 -1.5707" xyz="1.1385 0.0 -0.052"/>
+    <origin rpy="3.1416 0.0 -1.5707" xyz="0.4615 0.0 -0.052"/>
   </joint>
   <joint name="$(arg namespace)/camera_front_left_joint" type="fixed">
     <parent link="$(arg namespace)/base_link"/>
     <child link="$(arg namespace)/camera_front_left_link"/>
-    <origin rpy="1.3 3.1416 2.3416" xyz="1.313 0.048 -0.007"/>
+    <origin rpy="1.3 3.1416 2.3416" xyz="0.636 0.048 -0.007"/>
   </joint>
   <joint name="$(arg namespace)/camera_front_right_joint" type="fixed">
     <parent link="$(arg namespace)/base_link"/>
     <child link="$(arg namespace)/camera_front_right_link"/>
-    <origin rpy="1.3 3.1416 0.8" xyz="1.313 -0.048 -0.007"/>
+    <origin rpy="1.3 3.1416 0.8" xyz="0.636 -0.048 -0.007"/>
   </joint>
   <joint name="$(arg namespace)/lcg_joint" type="prismatic">
     <parent link="$(arg namespace)/base_link"/>
     <child link="$(arg namespace)/battery_link"/>
-    <origin rpy="0.0 0.0 0.0" xyz="0.76 0.0 0.0"/>
+    <origin rpy="0.0 0.0 0.0" xyz="0.083 0.0 0.0"/>
     <axis xyz="1 0 0"/>
     <limit lower="-0.01" upper="0.01" velocity="0.2" effort="1.0"/>
@@ -141,5 +141,5 @@
     <parent link="$(arg namespace)/base_link"/>
     <child link="$(arg namespace)/tcg1_link"/>
-    <origin rpy="0.0 0.0 0.0" xyz="0.582 0.0 0.0"/>
+    <origin rpy="0.0 0.0 0.0" xyz="-0.095 0.0 0.0"/>
     <axis xyz="1 0 0"/>
     <limit lower="-1.6" upper="1.6" velocity="0.2" effort="1.0"/>
@@ -148,5 +148,5 @@
     <parent link="$(arg namespace)/base_link"/>
     <child link="$(arg namespace)/tcg2_link"/>
-    <origin rpy="0.0 0.0 0.0" xyz="0.552 0.0 0.0"/>
+    <origin rpy="0.0 0.0 0.0" xyz="-0.125 0.0 0.0"/>
     <axis xyz="1 0 0"/>
     <limit lower="-1.6" upper="1.6" velocity="0.2" effort="1.0"/>

Commit message: Updated camera positions for waterlink nosecone

File: sam_description/urdf/sam_auv.urdf.xacro (robot description, xacro)
@@ -54,4 +54,5 @@
   <link name="$(arg namespace)/camera_front_right_link"/>
   <link name="$(arg namespace)/camera_front_left_link"/>
+  <link name="$(arg namespace)/camera_front_link"/>
   <joint name="$(arg namespace)/thruster_yaw_joint" type="revolute">
     <parent link="$(arg namespace)/base_link"/>
@@ -116,18 +117,25 @@
     <origin rpy="0.0 0.0 0.0" xyz="-0.402 0.0 0.078"/>
   </joint>
+  <!-- Waterlink Nosecone Camera Positions -->
+  <joint name="$(arg namespace)/camera_front_joint" type="fixed">
+    <parent link="$(arg namespace)/base_link"/>
+    <child link="$(arg namespace)/camera_front_link"/>
+    <origin rpy="0.0 1.5707 0.0" xyz="0.647 0.0 0.0"/>
+  </joint>
   <joint name="$(arg namespace)/camera_down_joint" type="fixed">
     <parent link="$(arg namespace)/base_link"/>
     <child link="$(arg namespace)/camera_down_link"/>
-    <origin rpy="3.1416 0.0 -1.5707" xyz="0.4615 0.0 -0.052"/>
+    <origin rpy="3.1416 0.0 -1.5707" xyz="0.5905 0.0 -0.058"/>
   </joint>
   <joint name="$(arg namespace)/camera_front_left_joint" type="fixed">
     <parent link="$(arg namespace)/base_link"/>
     <child link="$(arg namespace)/camera_front_left_link"/>
-    <origin rpy="1.3 3.1416 2.3416" xyz="0.636 0.048 -0.007"/>
+    <!--origin rpy="1.3 3.1416 2.3416" xyz="0.636 0.050 -0.007"/-->
+    <origin rpy="-0.2217 1.7243 0.6039" xyz="0.636 0.050 -0.007"/>
   </joint>
   <joint name="$(arg namespace)/camera_front_right_joint" type="fixed">
     <parent link="$(arg namespace)/base_link"/>
     <child link="$(arg namespace)/camera_front_right_link"/>
-    <origin rpy="1.3 3.1416 0.8" xyz="0.636 -0.048 -0.007"/>
+    <origin rpy="0.2217 1.7243 -0.6039" xyz="0.636 -0.050 -0.007"/>
   </joint>
   <joint name="$(arg namespace)/lcg_joint" type="prismatic">

Commit message: Latest cam defs. From David?

File: sam_description/urdf/sam_auv.urdf.xacro (robot description, xacro)
@@ -121,5 +121,5 @@
     <parent link="$(arg namespace)/base_link"/>
     <child link="$(arg namespace)/camera_front_link"/>
-    <origin rpy="0.0 1.5707 0.0" xyz="0.647 0.0 0.0"/>
+    <origin rpy="-1.5707 0.0 -1.5707" xyz="0.647 0.0 0.0"/>
   </joint>
   <joint name="$(arg namespace)/camera_down_joint" type="fixed">
@@ -132,10 +132,10 @@
     <child link="$(arg namespace)/camera_front_left_link"/>
     <!--origin rpy="1.3 3.1416 2.3416" xyz="0.636 0.050 -0.007"/-->
-    <origin rpy="-0.2217 1.7243 0.6039" xyz="0.636 0.050 -0.007"/>
+    <origin rpy="1.3 3.1416 2.3416" xyz="0.636 0.050 -0.007"/>
   </joint>
   <joint name="$(arg namespace)/camera_front_right_joint" type="fixed">
     <parent link="$(arg namespace)/base_link"/>
     <child link="$(arg namespace)/camera_front_right_link"/>
-    <origin rpy="0.2217 1.7243 -0.6039" xyz="0.636 -0.050 -0.007"/>
+    <origin rpy="1.3 3.1416 0.8" xyz="0.636 -0.050 -0.007"/>
   </joint>
   <joint name="$(arg namespace)/lcg_joint" type="prismatic">
