Commit message: Renames rtk links

File: floatsam_description/urdf/floatsam_usv.urdf.xacro (robot description, xacro)
@@ -19,6 +19,6 @@
   <link name="$(arg namespace)/gps_0_link"/>
   <link name="$(arg namespace)/gps_1_link"/>
-  <link name="$(arg namespace)/gps_2_link"/>
-  <link name="$(arg namespace)/gps_3_link"/>
+  <link name="$(arg namespace)/rtk_stb_link"/>
+  <link name="$(arg namespace)/rtk_prt_link"/>
   <link name="$(arg namespace)/uw_gps_link"/>
   <joint name="$(arg namespace)/thruster_port_joint" type="fixed">
@@ -52,12 +52,12 @@
     <origin rpy="0.0 0.0 0.0" xyz="0.5 -0.25 0.11"/>
   </joint>
-  <joint name="$(arg namespace)/gps_2_joint" type="fixed">
+  <joint name="$(arg namespace)/rtk_stb_joint" type="fixed">
     <parent link="$(arg namespace)/base_link"/>
-    <child link="$(arg namespace)/gps_2_link"/>
+    <child link="$(arg namespace)/rtk_stb_link"/>
     <origin rpy="0.0 0.0 0.0" xyz="-0.05 -0.25 0.11"/>
   </joint>
-  <joint name="$(arg namespace)/gps_3_joint" type="fixed">
+  <joint name="$(arg namespace)/rtk_prt_joint" type="fixed">
     <parent link="$(arg namespace)/base_link"/>
-    <child link="$(arg namespace)/gps_3_link"/>
+    <child link="$(arg namespace)/rtk_prt_link"/>
     <origin rpy="0.0 0.0 0.0" xyz="-0.05 0.25 0.11"/>
   </joint>

Commit message: Added DVL link

File: floatsam_description/urdf/floatsam_usv.urdf.xacro (robot description, xacro)
@@ -22,4 +22,5 @@
   <link name="$(arg namespace)/rtk_prt_link"/>
   <link name="$(arg namespace)/uw_gps_link"/>
+  <link name="$(arg namespace)/dvl_link"/>
   <joint name="$(arg namespace)/thruster_port_joint" type="fixed">
     <parent link="$(arg namespace)/base_link"/>
@@ -67,4 +68,9 @@
     <origin rpy="${PI} 0.0 ${PI / 2}" xyz="0.4 0. -0.15"/>
   </joint>
+  <joint name="$(arg namespace)/dvl_joint" type="fixed">
+    <parent link="$(arg namespace)/base_link"/>
+    <child link="$(arg namespace)/dvl_link"/>
+    <origin rpy="0. 0.0 0." xyz="0.42 -0.25 -0.15"/>
+  </joint>
   </xacro:macro>
 </robot>

Commit message: Added DVL link better pose

File: floatsam_description/urdf/floatsam_usv.urdf.xacro (robot description, xacro)
@@ -71,5 +71,5 @@
     <parent link="$(arg namespace)/base_link"/>
     <child link="$(arg namespace)/dvl_link"/>
-    <origin rpy="0. 0.0 0." xyz="0.42 -0.25 -0.15"/>
+    <origin rpy="0. 0.0 0." xyz="0.05 -0.25 -0.15"/>
   </joint>
   </xacro:macro>

Commit message: Latest UW GPS antenna pose

File: floatsam_description/urdf/floatsam_usv.urdf.xacro (robot description, xacro)
@@ -66,5 +66,5 @@
     <parent link="$(arg namespace)/base_link"/>
     <child link="$(arg namespace)/uw_gps_link"/>
-    <origin rpy="${PI} 0.0 ${PI / 2}" xyz="0.4 0. -0.15"/>
+    <origin rpy="${PI} 0.0 -${PI / 2}" xyz="0.4 0. -0.15"/>
   </joint>
   <joint name="$(arg namespace)/dvl_joint" type="fixed">
